File: PCB/gps_module.kicad_sch (KiCad schematic)
At the start: 0 parts

Commit message: Added connector for GPS
Parts:
- added J6: TEL0094, Connector_PinSocket_2.54mm:PinSocket_1x06_P2.54mm_Horizontal, symbol Connector_Generic:Conn_01x06
Connections:
- new net GND: J6.5 (Pin_5)
- new net GPS_EN: J6.6 (Pin_6)
- new net GPS_PPS: J6.1 (Pin_1)
- new net GPS_RX: J6.4 (Pin_4)
- new net GPS_TX: J6.3 (Pin_3)
- new net GPS_VCC_3V3: J6.2 (Pin_2)
Other:
- note added: "Still consider https://www.hestore.hu/prod_10041178.html# as an alternative the connector might not be suitable for extended usage in an environment with a lot of vibrations"
Changed lines of the file:
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@@
 (kicad_sch (version 20230121) (generator eeschema)
   (paper "A4")
+  (wire (pts (xy 199.39 78.74) (xy 204.47 78.74))
+    (stroke (width 0) (type default))
+  )
+  (wire (pts (xy 199.39 73.66) (xy 204.47 73.66))
+    (stroke (width 0) (type default))
+  )
+  (wire (pts (xy 199.39 66.04) (xy 204.47 66.04))
+    (stroke (width 0) (type default))
+  )
+  (wire (pts (xy 199.39 68.58) (xy 204.47 68.58))
+    (stroke (width 0) (type default))
+  )
+  (wire (pts (xy 185.42 76.2) (xy 185.42 77.47))
+    (stroke (width 0) (type default))
+  )
+  (wire (pts (xy 199.39 71.12) (xy 204.47 71.12))
+    (stroke (width 0) (type default))
+  )
+  (wire (pts (xy 204.47 76.2) (xy 185.42 76.2))
+    (stroke (width 0) (type default))
+  )
+  (text "Still consider https://www.hestore.hu/prod_10041178.html# as an alternative\nthe connector might not be suitable for extended usage in an environment with a lot of vibrations\n"
+    (at 228.6 53.34 0)
+    (effects (font (size 1.27 1.27)) (justify right bottom))
+  )
+  (global_label "GPS_EN" (shape passive) (at 199.39 78.74 180) (fields_autoplaced)
+    (effects (font (size 1.27 1.27)) (justify right))
+    (property "Intersheetrefs" "${INTERSHEET_REFS}" (at 190.3989 78.74 0)
+      (effects (font (size 1.27 1.27)) (justify right) hide)
+    )
+  )
+  (global_label "GPS_RX" (shape passive) (at 199.39 73.66 180) (fields_autoplaced)
+    (effects (font (size 1.27 1.27)) (justify right))
+    (property "Intersheetrefs" "${INTERSHEET_REFS}" (at 190.3989 73.66 0)
+      (effects (font (size 1.27 1.27)) (justify right) hide)
+    )
+  )
+  (global_label "GPS_VCC_3V3" (shape passive) (at 199.39 68.58 180) (fields_autoplaced)
+    (effects (font (size 1.27 1.27)) (justify right))
+    (property "Intersheetrefs" "${INTERSHEET_REFS}" (at 184.7746 68.58 0)
+      (effects (font (size 1.27 1.27)) (justify right) hide)
+    )
+  )
+  (global_label "GPS_PPS" (shape passive) (at 199.39 66.04 180) (fields_autoplaced)
+    (effects (font (size 1.27 1.27)) (justify right))
+    (property "Intersheetrefs" "${INTERSHEET_REFS}" (at 189.1289 66.04 0)
+      (effects (font (size 1.27 1.27)) (justify right) hide)
+    )
+  )
+  (global_label "GPS_TX" (shape passive) (at 199.39 71.12 180) (fields_autoplaced)
+    (effects (font (size 1.27 1.27)) (justify right))
+    (property "Intersheetrefs" "${INTERSHEET_REFS}" (at 190.7013 71.12 0)
+      (effects (font (size 1.27 1.27)) (justify right) hide)
+    )
+  )
+  (symbol (lib_id "Connector_Generic:Conn_01x06") (at 209.55 71.12 0) (unit 1)
+    (in_bom yes) (on_board yes) (dnp no) (fields_autoplaced)
+    (property "Reference" "J6" (at 212.09 71.755 0)
+      (effects (font (size 1.27 1.27)) (justify left))
+    )
+    (property "Value" "TEL0094" (at 212.09 74.295 0)
+      (effects (font (size 1.27 1.27)) (justify left))
+    )
+    (property "Footprint" "Connector_PinSocket_2.54mm:PinSocket_1x06_P2.54mm_Horizontal" (at 209.55 71.12 0)
+      (effects (font (size 1.27 1.27)) hide)
+    )
+    (property "Datasheet" "https://github.com/CainZ/V.KEL-GPS/raw/master/VK2828U7G5LF%20Data%20Sheet%2020150902.pdf" (at 209.55 71.12 0)
+      (effects (font (size 1.27 1.27)) hide)
+    )
+    (property "Farnell" "https://hu.farnell.com/dfrobot/tel0094/gps-3-3v-5v-56-ch-2-5m-ttl-uart/dp/3769993?st=gps" (at 209.55 71.12 0)
+      (effects (font (size 1.27 1.27)) hide)
+    )
+    (pin "1")
+    (pin "2")
+    (pin "3")
+    (pin "4")
+    (pin "5")
+    (pin "6")
+    (instances
+      (project "motor_tracker"
+        (path "/a8928dcf-7fea-46f0-8c15-a3fa49b43e6b/40317f30-d63d-4db0-91db-94d1ce3240f3"
+          (reference "J6") (unit 1)
+        )
+      )
+    )
+  )
+  (symbol (lib_id "power:GND") (at 185.42 77.47 0) (unit 1)
+    (in_bom yes) (on_board yes) (dnp no) (fields_autoplaced)
+    (property "Reference" "#PWR09" (at 185.42 83.82 0)
+      (effects (font (size 1.27 1.27)) hide)
+    )
+    (property "Value" "GND" (at 185.42 82.55 0)
+      (effects (font (size 1.27 1.27)))
+    )
+    (property "Footprint" "" (at 185.42 77.47 0)
+      (effects (font (size 1.27 1.27)) hide)
+    )
+    (property "Datasheet" "" (at 185.42 77.47 0)
+      (effects (font (size 1.27 1.27)) hide)
+    )
+    (pin "1")
+    (instances
+      (project "motor_tracker"
+        (path "/a8928dcf-7fea-46f0-8c15-a3fa49b43e6b/0c29d405-cd4c-45ef-9d08-777d8a682a5c"
+          (reference "#PWR09") (unit 1)
+        )
+        (path "/a8928dcf-7fea-46f0-8c15-a3fa49b43e6b/40317f30-d63d-4db0-91db-94d1ce3240f3"
+          (reference "#PWR022") (unit 1)
+        )
+      )
+    )
+  )
 )
