File: PCB/battery_management.kicad_sch (KiCad schematic)
At the start: 2 parts

Commit message: A bit of advancement in power and battery management
Parts:
- added J10: BatteryConnector, symbol Connector_Generic:Conn_01x04
Connections:
- new net BATTERY_PACK_C1+: J10.2 (Pin_2)
- new net BATTERY_PACK_C1-: J10.1 (Pin_1)
- new net BATTERY_PACK_C2+: J10.3 (Pin_3)
- new net BATTERY_PACK_C3+: J10.4 (Pin_4)
Other:
- moved on the sheet: R1
Changed lines of the file:
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@@
 (kicad_sch (version 20230121) (generator eeschema)
   (paper "A4")
-  (junction (at 31.75 41.91) (diameter 0) (color 0 0 0 0)
+  (junction (at 127 171.45) (diameter 0) (color 0 0 0 0)
   )
-  (wire (pts (xy 31.75 26.67) (xy 31.75 31.75))
+  (wire (pts (xy 130.81 157.48) (xy 127 157.48))
     (stroke (width 0) (type default))
   )
-  (wire (pts (xy 31.75 39.37) (xy 31.75 41.91))
+  (wire (pts (xy 27.94 21.59) (xy 30.48 21.59))
     (stroke (width 0) (type default))
   )
-  (wire (pts (xy 31.75 41.91) (xy 31.75 44.45))
+  (wire (pts (xy 27.94 29.21) (xy 30.48 29.21))
     (stroke (width 0) (type default))
   )
-  (wire (pts (xy 31.75 52.07) (xy 31.75 55.88))
+  (wire (pts (xy 27.94 24.13) (xy 30.48 24.13))
     (stroke (width 0) (type default))
   )
-  (wire (pts (xy 31.75 41.91) (xy 40.64 41.91))
+  (wire (pts (xy 127 168.91) (xy 127 171.45))
     (stroke (width 0) (type default))
   )
-  (global_label "VCC_INTERNAL_BATTERY" (shape passive) (at 31.75 26.67 0) (fields_autoplaced)
+  (wire (pts (xy 127 171.45) (xy 127 173.99))
+    (stroke (width 0) (type default))
+  )
+  (wire (pts (xy 127 157.48) (xy 127 161.29))
+    (stroke (width 0) (type default))
+  )
+  (wire (pts (xy 27.94 26.67) (xy 30.48 26.67))
+    (stroke (width 0) (type default))
+  )
+  (wire (pts (xy 127 181.61) (xy 127 185.42))
+    (stroke (width 0) (type default))
+  )
+  (wire (pts (xy 127 171.45) (xy 139.7 171.45))
+    (stroke (width 0) (type default))
+  )
+  (global_label "BATTERY_PACK_C1+" (shape passive) (at 30.48 26.67 0) (fields_autoplaced)
     (effects (font (size 1.27 1.27)) (justify left))
-    (property "Intersheetrefs" "${INTERSHEET_REFS}" (at 55.6788 26.67 0)
+    (property "Intersheetrefs" "${INTERSHEET_REFS}" (at 50.9616 26.67 0)
       (effects (font (size 1.27 1.27)) (justify left) hide)
     )
   )
-  (global_label "VCC_INPUT_A" (shape passive) (at 40.64 41.91 0) (fields_autoplaced)
+  (global_label "BATTERY_PACK_C1-" (shape passive) (at 30.48 29.21 0) (fields_autoplaced)
     (effects (font (size 1.27 1.27)) (justify left))
-    (property "Intersheetrefs" "${INTERSHEET_REFS}" (at 54.5903 41.91 0)
+    (property "Intersheetrefs" "${INTERSHEET_REFS}" (at 50.9616 29.21 0)
       (effects (font (size 1.27 1.27)) (justify left) hide)
     )
   )
-  (symbol (lib_id "power:GND") (at 31.75 55.88 0) (unit 1)
+  (global_label "BATTERY_PACK_C2+" (shape passive) (at 30.48 24.13 0) (fields_autoplaced)
+    (effects (font (size 1.27 1.27)) (justify left))
+    (property "Intersheetrefs" "${INTERSHEET_REFS}" (at 50.9616 24.13 0)
+      (effects (font (size 1.27 1.27)) (justify left) hide)
+    )
+  )
+  (global_label "VCC_INTERNAL_BATTERY" (shape passive) (at 238.76 29.21 0) (fields_autoplaced)
+    (effects (font (size 1.27 1.27)) (justify left))
+    (property "Intersheetrefs" "${INTERSHEET_REFS}" (at 262.6888 29.21 0)
+      (effects (font (size 1.27 1.27)) (justify left) hide)
+    )
+  )
+  (global_label "VCC_INTERNAL_BATTERY" (shape passive) (at 130.81 157.48 0) (fields_autoplaced)
+    (effects (font (size 1.27 1.27)) (justify left))
+    (property "Intersheetrefs" "${INTERSHEET_REFS}" (at 154.7388 157.48 0)
+      (effects (font (size 1.27 1.27)) (justify left) hide)
+    )
+  )
+  (global_label "VCC_INPUT_A" (shape passive) (at 139.7 171.45 0) (fields_autoplaced)
+    (effects (font (size 1.27 1.27)) (justify left))
+    (property "Intersheetrefs" "${INTERSHEET_REFS}" (at 153.6503 171.45 0)
+      (effects (font (size 1.27 1.27)) (justify left) hide)
+    )
+  )
+  (global_label "BATTERY_PACK_C3+" (shape passive) (at 30.48 21.59 0) (fields_autoplaced)
+    (effects (font (size 1.27 1.27)) (justify left))
+    (property "Intersheetrefs" "${INTERSHEET_REFS}" (at 50.9616 21.59 0)
+      (effects (font (size 1.27 1.27)) (justify left) hide)
+    )
+  )
+  (symbol (lib_id "power:GND") (at 127 185.42 0) (unit 1)
     (in_bom yes) (on_board yes) (dnp no) (fields_autoplaced)
-    (property "Reference" "#PWR02" (at 31.75 62.23 0)
+    (property "Reference" "#PWR02" (at 127 191.77 0)
       (effects (font (size 1.27 1.27)) hide)
     )
-    (property "Value" "GND" (at 31.75 60.96 0)
+    (property "Value" "GND" (at 127 190.5 0)
       (effects (font (size 1.27 1.27)))
     )
-    (property "Footprint" "" (at 31.75 55.88 0)
+    (property "Footprint" "" (at 127 185.42 0)
       (effects (font (size 1.27 1.27)) hide)
     )
-    (property "Datasheet" "" (at 31.75 55.88 0)
+    (property "Datasheet" "" (at 127 185.42 0)
       (effects (font (size 1.27 1.27)) hide)
     )
@@
     )
   )
-  (symbol (lib_id "Device:R") (at 31.75 48.26 180) (unit 1)
+  (symbol (lib_id "Device:R") (at 127 177.8 180) (unit 1)
     (in_bom yes) (on_board yes) (dnp no) (fields_autoplaced)
-    (property "Reference" "R1" (at 34.29 47.625 0)
+    (property "Reference" "R1" (at 129.54 177.165 0)
       (effects (font (size 1.27 1.27)) (justify right))
     )
-    (property "Value" "110k" (at 34.29 50.165 0)
+    (property "Value" "110k" (at 129.54 179.705 0)
       (effects (font (size 1.27 1.27)) (justify right))
     )
-    (property "Footprint" "Resistor_SMD:R_0603_1608Metric_Pad0.98x0.95mm_HandSolder" (at 33.528 48.26 90)
+    (property "Footprint" "Resistor_SMD:R_0603_1608Metric_Pad0.98x0.95mm_HandSolder" (at 128.778 177.8 90)
       (effects (font (size 1.27 1.27)) hide)
     )
-    (property "Datasheet" "~" (at 31.75 48.26 0)
+    (property "Datasheet" "~" (at 127 177.8 0)
       (effects (font (size 1.27 1.27)) hide)
     )
@@
     )
   )
-  (symbol (lib_id "Device:R") (at 31.75 35.56 180) (unit 1)
+  (symbol (lib_id "Device:R") (at 127 165.1 180) (unit 1)
     (in_bom yes) (on_board yes) (dnp no) (fields_autoplaced)
-    (property "Reference" "R1" (at 34.29 34.925 0)
+    (property "Reference" "R1" (at 129.54 164.465 0)
       (effects (font (size 1.27 1.27)) (justify right))
     )
-    (property "Value" "620k" (at 34.29 37.465 0)
+    (property "Value" "620k" (at 129.54 167.005 0)
       (effects (font (size 1.27 1.27)) (justify right))
     )
-    (property "Footprint" "Resistor_SMD:R_0603_1608Metric_Pad0.98x0.95mm_HandSolder" (at 33.528 35.56 90)
+    (property "Footprint" "Resistor_SMD:R_0603_1608Metric_Pad0.98x0.95mm_HandSolder" (at 128.778 165.1 90)
       (effects (font (size 1.27 1.27)) hide)
     )
-    (property "Datasheet" "~" (at 31.75 35.56 0)
+    (property "Datasheet" "~" (at 127 165.1 0)
       (effects (font (size 1.27 1.27)) hide)
     )
@@
         )
       )
+    )
+  )
+  (symbol (lib_id "Connector_Generic:Conn_01x04") (at 22.86 26.67 180) (unit 1)
+    (in_bom yes) (on_board yes) (dnp no) (fields_autoplaced)
+    (property "Reference" "J10" (at 22.86 16.51 0)
+      (effects (font (size 1.27 1.27)))
+    )
+    (property "Value" "BatteryConnector" (at 22.86 19.05 0)
+      (effects (font (size 1.27 1.27)))
+    )
+    (property "Footprint" "" (at 22.86 26.67 0)
+      (effects (font (size 1.27 1.27)) hide)
+    )
+    (property "Datasheet" "~" (at 22.86 26.67 0)
+      (effects (font (size 1.27 1.27)) hide)
+    )
+    (pin "1")
+    (pin "2")
+    (pin "3")
+    (pin "4")
+    (instances
+      (project "motor_tracker"
+        (path "/a8928dcf-7fea-46f0-8c15-a3fa49b43e6b/00a7dfb5-f91b-41af-916a-3d945a79f238"
+          (reference "J10") (unit 1)
+        )
+      )
